File: hardware/gnss-module/gnss-module.kicad_pcb (KiCad board)
At the start: 4 copper layers, 89.1 x 92.2 mm, 21 parts, among them J1 Conn_01x04_Pin, J2 Conn_01x04_Pin, J3 USB_B_Micro, J4 Conn_01x02_Pin, J5 Conn_01x20_Socket, J6 Conn_01x04_Pin, U1 LM1117MP-ADJ

Commit message: main: Socket connector changed
Parts:
- J5: footprint Connector_PinSocket_2.00mm:PinSocket_2x10_P2.00mm_Vertical_SMD -> spacelab_lib:SAMTEC-SQW-110-01-X-D
- turned J5 to 180 degrees
Routing:
- net /TXD2: track 42.1 -> 48.7 mm, vias 0 -> 1
- net /D2_P: track 22.3 -> 16.6 mm
- net /3V3: track 13.8 -> 9.25 mm, vias 6 -> 4
- net /D2_N: track 22.3 -> 18.2 mm
- net /RXD1: track 39.6 -> 38.2 mm
- net /TXD1: track 39.5 -> 40.5 mm
- net /RXD2: track 50.3 -> 50.1 mm, vias 2 -> 1

Commit message: main: Socket connector changed
Parts:
- J5: footprint spacelab_lib:SAMTEC-SQW-110-01-X-D -> spacelab_lib:SAMTEC-SQW-110-01-X-D-VS
- moved L2 5.53 mm to (399.3, 310.7)
- moved D2 2.23 mm to (403.7, 311.0), turned to -45 degrees
Connections:
- D2 pad 1: /D1_N -> /D1_P
- D2 pad 2: /D1_P -> /D1_N
Routing:
- net /D2_P: track 16.6 -> 24.6 mm
- net /D2_N: track 18.2 -> 24.6 mm
- net /D1_P: track 14.0 -> 8.30 mm
- net /D1_N: track 13.6 -> 8.34 mm
- net /TXD2: track 48.7 -> 44.1 mm, vias 1 -> 2
- net /TXD1: track 40.5 -> 45.0 mm
- net /3V3: track 9.25 -> 13.1 mm, vias 4 -> 6
- net /RXD2: track 50.1 -> 51.3 mm, vias 1 -> 2
