File: hardware/gnss-module/gnss-module.kicad_sch (KiCad schematic)
At the start: 21 parts, among them J1 Conn_01x04_Pin, J2 Conn_01x04_Pin, J3 USB_B_Micro, J4 Conn_01x02_Pin, J5 Conn_01x20_Socket, J6 Conn_01x04_Pin, U1 LM1117MP-ADJ

Commit message: main: Socket connector changed
Parts:
- J5: footprint Connector_PinSocket_2.00mm:PinSocket_2x10_P2.00mm_Vertical_SMD -> spacelab_lib:SAMTEC-SQW-110-01-X-D

Commit message: main: Socket connector changed
Parts:
- J5: footprint spacelab_lib:SAMTEC-SQW-110-01-X-D -> spacelab_lib:SAMTEC-SQW-110-01-X-D-VS
Connections:
- net D1_N: now also D2.2 (K); no longer D2.1 (K)
- net D1_P: now also D2.1 (K); no longer D2.2 (K)
Changed lines of the file:
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@@
 	)
 	(junction
-		(at 71.12 38.1)
+		(at 182.88 86.36)
 		(diameter 0)
 		(color 0 0 0 0)
 	)
 	(junction
-		(at 106.68 38.1)
+		(at 187.96 83.82)
 		(diameter 0)
 		(color 0 0 0 0)
 	)
 	(junction
-		(at 182.88 86.36)
+		(at 71.12 38.1)
+		(diameter 0)
+		(color 0 0 0 0)
+	)
+	(junction
+		(at 106.68 38.1)
 		(diameter 0)
 		(color 0 0 0 0)
@@
 	)
 	(junction
-		(at 187.96 83.82)
-		(diameter 0)
-		(color 0 0 0 0)
-	)
-	(junction
 		(at 121.92 46.99)
 		(diameter 0)
@@
 	(wire
 		(pts
-			(xy 182.88 86.36) (xy 182.88 91.44)
+			(xy 83.82 50.8) (xy 83.82 48.26)
 		)
 		(stroke
@@
 	(wire
 		(pts
-			(xy 83.82 50.8) (xy 83.82 48.26)
+			(xy 182.88 86.36) (xy 182.88 91.44)
 		)
 		(stroke
@@
 	(wire
 		(pts
-			(xy 182.88 86.36) (xy 214.63 86.36)
+			(xy 256.54 144.78) (xy 256.54 142.24)
 		)
 		(stroke
@@
 	(wire
 		(pts
-			(xy 256.54 144.78) (xy 256.54 142.24)
+			(xy 251.46 144.78) (xy 256.54 144.78)
 		)
 		(stroke
@@
 	(wire
 		(pts
-			(xy 251.46 144.78) (xy 256.54 144.78)
+			(xy 41.91 121.92) (xy 35.56 121.92)
 		)
 		(stroke
@@
 	(wire
 		(pts
-			(xy 41.91 121.92) (xy 35.56 121.92)
+			(xy 83.82 40.64) (xy 83.82 38.1)
 		)
 		(stroke
@@
 	(wire
 		(pts
-			(xy 83.82 40.64) (xy 83.82 38.1)
+			(xy 129.54 38.1) (xy 134.62 38.1)
 		)
 		(stroke
@@
 	(wire
 		(pts
-			(xy 129.54 38.1) (xy 134.62 38.1)
+			(xy 182.88 86.36) (xy 214.63 86.36)
 		)
 		(stroke
@@
 	(wire
 		(pts
-			(xy 187.96 83.82) (xy 187.96 91.44)
-		)
-		(stroke
-			(width 0)
-			(type default)
-		)
-	)
-	(wire
-		(pts
 			(xy 134.62 45.72) (xy 134.62 46.99)
 		)
@@
 	(wire
 		(pts
+			(xy 187.96 83.82) (xy 187.96 91.44)
+		)
+		(stroke
+			(width 0)
+			(type default)
+		)
+	)
+	(wire
+		(pts
 			(xy 41.91 137.16) (xy 35.56 137.16)
 		)
@@
 			)
 		)
-		(property "Footprint" "spacelab_lib:SAMTEC-SQW-110-01-X-D"
+		(property "Footprint" "spacelab_lib:SAMTEC-SQW-110-01-X-D-VS"
 			(at 30.48 147.32 0)
 			(effects
@@
 		(lib_id "Power_Protection:NUP2105L")
 		(at 185.42 96.52 0)
-		(mirror y)
 		(unit 1)
 		(exclude_from_sim no)
@@
 		(dnp no)
 		(property "Reference" "D2"
-			(at 179.07 95.2499 0)
+			(at 191.77 95.2499 0)
 			(effects
 				(font
@@
 		)
 		(property "Value" "NUP2105L"
-			(at 179.07 97.7899 0)
+			(at 191.77 97.7899 0)
 			(effects
 				(font
@@
 		)
 		(property "Footprint" "spacelab_lib:SOT-723_0P85X1P25_ONS-M"
-			(at 179.705 97.79 0)
+			(at 191.135 97.79 0)
 			(effects
 				(font
@@
 		)
 		(property "Datasheet" "https://www.onsemi.com/pub_link/Collateral/NUP2105L-D.PDF"
-			(at 182.245 93.345 0)
+			(at 188.595 93.345 0)
 			(effects
 				(font
