File: hardware/_autosave-gnss_pod.kicad_pcb (KiCad board)
At the start: 2 copper layers, 240.3 x 213.8 mm, 19 parts, among them J1 SQT-110-01-L-D, J2 SSQ-126-04-G-D, J3 SSQ-126-04-G-D

Commit message: Updated layout + schematic
Parts:
- H1, H2, H3, H4, H5, H6, H7, H8: footprint MountingHole:MountingHole_6mm_Pad -> MountingHole:MountingHole_3mm_Pad
Changed lines of the file:
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@@
 		(embedded_fonts no)
 	)
-	(footprint "MountingHole:MountingHole_6mm_Pad"
+	(footprint "MountingHole:MountingHole_3mm_Pad"
 		(layer "F.Cu")
 		(at 306.65 128.8)
-		(descr "Mounting Hole 6mm, generated by kicad-footprint-generator mountinghole.py")
+		(descr "Mounting Hole 3mm, generated by kicad-footprint-generator mountinghole.py")
 		(tags "mountinghole")
 		(property "Reference" "H2"
-			(at 0 -6.95 0)
+			(at 0 -3.95 0)
 			(layer "F.SilkS")
 			(effects
@@
 		)
 		(property "Value" "MountingHole"
-			(at 0 6.95 0)
+			(at 0 3.95 0)
 			(layer "F.Fab")
 			(effects
@@
 		(fp_circle
 			(center 0 0)
-			(end 6 0)
+			(end 3 0)
 			(stroke
 				(width 0.15)
@@
 		(fp_circle
 			(center 0 0)
-			(end 6.25 0)
+			(end 3.25 0)
 			(stroke
 				(width 0.05)
@@
 		(pad "1" thru_hole circle
 			(at 0 0)
-			(size 12 12)
-			(drill 6)
+			(size 6 6)
+			(drill 3)
 			(layers "*.Cu" "*.Mask")
 			(remove_unused_layers no)
@@
 		(embedded_fonts no)
 	)
-	(footprint "MountingHole:MountingHole_6mm_Pad"
+	(footprint "MountingHole:MountingHole_3mm_Pad"
 		(layer "F.Cu")
 		(at 347.3 115.25)
-		(descr "Mounting Hole 6mm, generated by kicad-footprint-generator mountinghole.py")
+		(descr "Mounting Hole 3mm, generated by kicad-footprint-generator mountinghole.py")
 		(tags "mountinghole")
 		(property "Reference" "H7"
-			(at 0 -6.95 0)
+			(at 0 -3.95 0)
 			(layer "F.SilkS")
 			(effects
@@
 		)
 		(property "Value" "MountingHole"
-			(at 0 6.95 0)
+			(at 0 3.95 0)
 			(layer "F.Fab")
 			(effects
@@
 		(fp_circle
 			(center 0 0)
-			(end 6 0)
+			(end 3 0)
 			(stroke
 				(width 0.15)
@@
 		(fp_circle
 			(center 0 0)
-			(end 6.25 0)
+			(end 3.25 0)
 			(stroke
 				(width 0.05)
@@
 		(pad "1" thru_hole circle
 			(at 0 0)
-			(size 12 12)
-			(drill 6)
+			(size 6 6)
+			(drill 3)
 			(layers "*.Cu" "*.Mask")
 			(remove_unused_layers no)
@@
 		(embedded_fonts no)
 	)
-	(footprint "MountingHole:MountingHole_6mm_Pad"
+	(footprint "MountingHole:MountingHole_3mm_Pad"
 		(layer "F.Cu")
 		(at 320.2 115.25)
-		(descr "Mounting Hole 6mm, generated by kicad-footprint-generator mountinghole.py")
+		(descr "Mounting Hole 3mm, generated by kicad-footprint-generator mountinghole.py")
 		(tags "mountinghole")
 		(property "Reference" "H3"
-			(at 0 -6.95 0)
+			(at 0 -3.95 0)
 			(layer "F.SilkS")
 			(effects
@@
 		)
 		(property "Value" "MountingHole"
-			(at 0 6.95 0)
+			(at 0 3.95 0)
 			(layer "F.Fab")
 			(effects
@@
 		(fp_circle
 			(center 0 0)
-			(end 6 0)
+			(end 3 0)
 			(stroke
 				(width 0.15)
@@
 		(fp_circle
 			(center 0 0)
-			(end 6.25 0)
+			(end 3.25 0)
 			(stroke
 				(width 0.05)
@@
 		(pad "1" thru_hole circle
 			(at 0 0)
-			(size 12 12)
-			(drill 6)
+			(size 6 6)
+			(drill 3)
 			(layers "*.Cu" "*.Mask")
 			(remove_unused_layers no)
@@
 		(embedded_fonts no)
 	)
-	(footprint "MountingHole:MountingHole_6mm_Pad"
+	(footprint "MountingHole:MountingHole_3mm_Pad"
 		(layer "F.Cu")
 		(at 333.75 128.8)
-		(descr "Mounting Hole 6mm, generated by kicad-footprint-generator mountinghole.py")
+		(descr "Mounting Hole 3mm, generated by kicad-footprint-generator mountinghole.py")
 		(tags "mountinghole")
 		(property "Reference" "H6"
-			(at 0 -6.95 0)
+			(at 0 -3.95 0)
 			(layer "F.SilkS")
 			(effects
@@
 		)
 		(property "Value" "MountingHole"
-			(at 0 6.95 0)
+			(at 0 3.95 0)
 			(layer "F.Fab")
 			(effects
@@
 		(fp_circle
 			(center 0 0)
-			(end 6 0)
+			(end 3 0)
 			(stroke
 				(width 0.15)
@@
 		(fp_circle
 			(center 0 0)
-			(end 6.25 0)
+			(end 3.25 0)
 			(stroke
 				(width 0.05)
@@
 		(pad "1" thru_hole circle
 			(at 0 0)
-			(size 12 12)
-			(drill 6)
+			(size 6 6)
+			(drill 3)
 			(layers "*.Cu" "*.Mask")
 			(remove_unused_layers no)
@@
 		)
 	)
-	(footprint "MountingHole:MountingHole_6mm_Pad"
+	(footprint "MountingHole:MountingHole_3mm_Pad"
 		(layer "F.Cu")
 		(at 320.2 128.8)
-		(descr "Mounting Hole 6mm, generated by kicad-footprint-generator mountinghole.py")
+		(descr "Mounting Hole 3mm, generated by kicad-footprint-generator mountinghole.py")
 		(tags "mountinghole")
 		(property "Reference" "H4"
-			(at 0 -6.95 0)
+			(at 0 -3.95 0)
 			(layer "F.SilkS")
 			(effects
@@
 		)
 		(property "Value" "MountingHole"
-			(at 0 6.95 0)
+			(at 0 3.95 0)
 			(layer "F.Fab")
 			(effects
@@
 		(fp_circle
 			(center 0 0)
-			(end 6 0)
+			(end 3 0)
 			(stroke
 				(width 0.15)
@@
 		(fp_circle
 			(center 0 0)
-			(end 6.25 0)
+			(end 3.25 0)
 			(stroke
 				(width 0.05)
@@
 		(pad "1" thru_hole circle
 			(at 0 0)
-			(size 12 12)
-			(drill 6)
+			(size 6 6)
+			(drill 3)
 			(layers "*.Cu" "*.Mask")
 			(remove_unused_layers no)
@@
 		(embedded_fonts no)
 	)
-	(footprint "MountingHole:MountingHole_6mm_Pad"
+	(footprint "MountingHole:MountingHole_3mm_Pad"
 		(layer "F.Cu")
 		(at 347.3 128.8)
-		(descr "Mounting Hole 6mm, generated by kicad-footprint-generator mountinghole.py")
+		(descr "Mounting Hole 3mm, generated by kicad-footprint-generator mountinghole.py")
 		(tags "mountinghole")
 		(property "Reference" "H8"
-			(at 0 -6.95 0)
+			(at 0 -3.95 0)
 			(layer "F.SilkS")
 			(effects
@@
 		)
 		(property "Value" "MountingHole"
-			(at 0 6.95 0)
+			(at 0 3.95 0)
 			(layer "F.Fab")
 			(effects
@@
 		(fp_circle
 			(center 0 0)
-			(end 6 0)
+			(end 3 0)
 			(stroke
 				(width 0.15)
@@
 		(fp_circle
 			(center 0 0)
-			(end 6.25 0)
+			(end 3.25 0)
 			(stroke
 				(width 0.05)
@@
 		(pad "1" thru_hole circle
 			(at 0 0)
-			(size 12 12)
-			(drill 6)
+			(size 6 6)
+			(drill 3)
 			(layers "*.Cu" "*.Mask")
 			(remove_unused_layers no)
@@
 		(embedded_fonts no)
 	)
-	(footprint "MountingHole:MountingHole_6mm_Pad"
+	(footprint "MountingHole:MountingHole_3mm_Pad"
 		(layer "F.Cu")
 		(at 306.65 115.25)
-		(descr "Mounting Hole 6mm, generated by kicad-footprint-generator mountinghole.py")
+		(descr "Mounting Hole 3mm, generated by kicad-footprint-generator mountinghole.py")
 		(tags "mountinghole")
 		(property "Reference" "H1"
-			(at 0 -6.95 0)
+			(at 0 -3.95 0)
 			(layer "F.SilkS")
 			(effects
@@
 		)
 		(property "Value" "MountingHole"
-			(at 0 6.95 0)
+			(at 0 3.95 0)
 			(layer "F.Fab")
 			(effects
@@
 		(fp_circle
 			(center 0 0)
-			(end 6 0)
+			(end 3 0)
 			(stroke
 				(width 0.15)
@@
 		(fp_circle
 			(center 0 0)
-			(end 6.25 0)
+			(end 3.25 0)
 			(stroke
 				(width 0.05)
@@
 		(pad "1" thru_hole circle
 			(at 0 0)
-			(size 12 12)
-			(drill 6)
+			(size 6 6)
+			(drill 3)
 			(layers "*.Cu" "*.Mask")
 			(remove_unused_layers no)
@@
 		(embedded_fonts no)
 	)
-	(footprint "MountingHole:MountingHole_6mm_Pad"
+	(footprint "MountingHole:MountingHole_3mm_Pad"
 		(layer "F.Cu")
 		(at 333.75 115.25)
-		(descr "Mounting Hole 6mm, generated by kicad-footprint-generator mountinghole.py")
+		(descr "Mounting Hole 3mm, generated by kicad-footprint-generator mountinghole.py")
 		(tags "mountinghole")
 		(property "Reference" "H5"
-			(at 0 -6.95 0)
+			(at 0 -3.95 0)
 			(layer "F.SilkS")
 			(effects
@@
 		)
 		(property "Value" "MountingHole"
-			(at 0 6.95 0)
+			(at 0 3.95 0)
 			(layer "F.Fab")
 			(effects
@@
 		(fp_circle
 			(center 0 0)
-			(end 6 0)
+			(end 3 0)
 			(stroke
 				(width 0.15)
@@
 		(fp_circle
 			(center 0 0)
-			(end 6.25 0)
+			(end 3.25 0)
 			(stroke
 				(width 0.05)
@@
 		(pad "1" thru_hole circle
 			(at 0 0)
-			(size 12 12)
-			(drill 6)
+			(size 6 6)
+			(drill 3)
 			(layers "*.Cu" "*.Mask")
 			(remove_unused_layers no)
