File: hardware/gnss_pod.kicad_sch (KiCad schematic)
At the start: 14 parts, among them J1 SQT-110-01-L-D, J2 SSQ-126-04-G-D, J3 SSQ-126-04-G-D, J4 Conn_01x02_Pin, J5 Conn_01x02_Pin, J6 USB_C_Receptacle_USB2.0_16P

Commit message: Trace match, PC104 adjusted, Hole Diameter.
- PC104 was mirrored;
- USB Trace is match by less then 1mm;
- CAN is not trace matched;
- Adjusted hole diameter for OEM719 Receiver (3mm -> 3.45mm);
- Trace is bigger for VCC.
Parts:
- added FB3: FerriteBead_Small, Inductor_SMD:L_0603_1608Metric, symbol Device:FerriteBead_Small
- added R3, R4: 5K1, Resistor_SMD:R_0603_1608Metric, symbol Device:R_Small_US
- renumbered J3 to J2, J2 to J3
Connections:
- net GNDREF: now also FB3.2, R3.2, R4.2
- net RX1: now also J2.19; no longer J3.19
- net TX1: now also J2.17; no longer J3.17
- net VCC: now also J3.35, J3.36; no longer J2.35, J2.36
- net at J6.A5 (CC1): now also R3.1
- net at J6.B5 (CC2): now also R4.1
- net at J6.SH (SHIELD): now also FB3.1
- no-connect marks 105 -> 102
Other:
- note added: "3 mm"
- note added: "3.45 mm"
- note added: "CAN (ESD)"
- note added: "H1"
- note added: "H2"
- note added: "P1701"
- note added: "PC104"
- note added: "UART"
- note added: "USB 2.0 Type - C"
- note removed: "<- REVISAR!"
- moved on the sheet: J2, J3, J4, J5, J6
