File: hardware/holder_can.kicad_sch (KiCad schematic)
At the start: 9 parts, among them IC1 CDNBS08-PLC03-6, U1 TCAN334G

Commit message: Added some connections, infos and USB footprint
Parts:
- FB1, FB2: footprint (none) -> Inductor_SMD:L_0402_1005Metric_Pad0.77x0.64mm_HandSolder
Changed lines of the file:
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@@
 			)
 		)
-		(property "Footprint" ""
+		(property "Footprint" "Inductor_SMD:L_0402_1005Metric_Pad0.77x0.64mm_HandSolder"
 			(at 138.43 89.408 90)
 			(hide yes)
@@
 			)
 		)
-		(property "Footprint" ""
+		(property "Footprint" "Inductor_SMD:L_0402_1005Metric_Pad0.77x0.64mm_HandSolder"
 			(at 138.43 109.728 90)
 			(hide yes)

Commit message: Receiver Flipped, Added Simple Match lenght traces, Added more silkscreen comments
Other:
- note added: "ESD Protection"
Changed lines of the file:
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@@
 		(company "SpaceLab")
+	)
+	(rectangle
+		(start 123.19 78.994)
+		(end 231.14 116.332)
+		(stroke
+			(width 0)
+			(type default)
+		)
+		(fill
+			(type none)
+		)
+	)
+	(text "ESD Protection"
+		(exclude_from_sim no)
+		(at 130.048 77.978 0)
+		(effects
+			(font
+				(size 1.27 1.27)
+				(thickness 0.254)
+				(bold yes)
+			)
+		)
 	)
 	(junction

Commit message: Trace match, PC104 adjusted, Hole Diameter.
- PC104 was mirrored;
- USB Trace is match by less then 1mm;
- CAN is not trace matched;
- Adjusted hole diameter for OEM719 Receiver (3mm -> 3.45mm);
- Trace is bigger for VCC.
Changed lines of the file:
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@@
 	(title_block
 		(title "GNSS POD - HOLDER")
-		(date "2026-07-21")
+		(date "2026-09-10")
 		(rev "0.1.0")
 		(company "SpaceLab")
+		(comment 2 "Arthur F. De S. Filho <Arthur-filho@live.com>")
+		(comment 3 "João V. Perin <Joaoperin.ufsc@gmail.com>")
 	)
 	(rectangle
 		(start 123.19 78.994)
-		(end 231.14 116.332)
+		(end 219.202 116.332)
 		(stroke
 			(width 0)
