File: hardware/GNSS_POD_PROT.kicad_pcb (KiCad board)
At the start: 2 copper layers, 34 x 18 mm, 3 parts, among them J1 Conn_01x02_Pin, J2 Conn_01x02_Pin, J3 SQT-110-01-L-D

Commit message: Fix track face and size
Parts:
- moved J3 7.28 mm to (128.3, 83.4)
Routing:
- net /RX1: track 23.2 -> 30.6 mm
- net /TX1: track 9.02 -> 16.3 mm
- net VCC: track 13.3 -> 20.5 mm
Other:
- board size 34 x 18 mm -> 34 x 24.8 mm
Changed lines of the file:
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@@
 		(capping no)
 		(filling no)
+		(zone_defaults)
 		(pcbplotparams
 			(layerselection 0x00000000_00000000_55555555_5755f5ff)
@@
 	(footprint "footprints:SQT11001LD"
 		(layer "F.Cu")
-		(at 128.3 76.125 180)
+		(at 128.3 83.4 180)
 		(descr "SQT-110-01-L-D-11")
 		(tags "Connector")
@@
 	)
 	(gr_line
-		(start 148.3 74.15)
-		(end 148.3 71.25)
-		(stroke
-			(width 0.1)
-			(type default)
-		)
-		(layer "F.SilkS")
-	)
-	(gr_line
 		(start 114.5 145.55)
 		(end 114.5 74.45)
@@
 	(gr_rect
 		(start 120.2 65.25)
-		(end 154.2 83.25)
+		(end 154.2 90)
 		(stroke
 			(width 0.2)
@@
 	)
 	(segment
-		(start 128.09 69.45)
+		(start 124.245 83.57)
 		(end 124.245 73.295)
 		(width 0.8)
-		(layer "F.Cu")
+		(layer "B.Cu")
 		(net "VCC")
 	)
 	(segment
-		(start 124.245 76.295)
-		(end 124.245 73.295)
+		(start 124.245 73.295)
+		(end 128.09 69.45)
 		(width 0.8)
-		(layer "F.Cu")
+		(layer "B.Cu")
 		(net "VCC")
 	)
 	(segment
-		(start 124.7 76.75)
-		(end 124.245 76.295)
+		(start 126.075 85.4)
+		(end 124.245 83.57)
 		(width 0.8)
-		(layer "F.Cu")
+		(layer "B.Cu")
 		(net "VCC")
 	)
 	(segment
-		(start 128.3 78.125)
-		(end 126.075 78.125)
+		(start 128.3 85.4)
+		(end 126.075 85.4)
 		(width 0.8)
-		(layer "F.Cu")
-		(net "VCC")
-	)
-	(segment
-		(start 126.075 78.125)
-		(end 124.7 76.75)
-		(width 0.8)
-		(layer "F.Cu")
+		(layer "B.Cu")
 		(net "VCC")
 	)
 	(segment
 		(start 138.3 75.1)
-		(end 138.3 76.125)
-		(width 0.3)
-		(layer "F.Cu")
+		(end 138.3 83.4)
+		(width 0.508)
+		(layer "B.Cu")
 		(net "/TX1")
 	)
@@
 		(start 143.95 69.45)
 		(end 138.3 75.1)
-		(width 0.3)
-		(layer "F.Cu")
+		(width 0.508)
+		(layer "B.Cu")
 		(net "/TX1")
+	)
+	(segment
+		(start 149.2 86.1)
+		(end 147.2 88.1)
+		(width 0.508)
+		(layer "B.Cu")
+		(net "/RX1")
+	)
+	(segment
+		(start 149.2 72.16)
+		(end 149.2 86.1)
+		(width 0.508)
+		(layer "B.Cu")
+		(net "/RX1")
 	)
 	(segment
 		(start 146.49 69.45)
 		(end 149.2 72.16)
-		(width 0.3)
-		(layer "F.Cu")
+		(width 0.508)
+		(layer "B.Cu")
 		(net "/RX1")
 	)
 	(segment
-		(start 149.2 72.16)
-		(end 149.2 78.75)
-		(width 0.3)
-		(layer "F.Cu")
+		(start 140.925 88.1)
+		(end 138.3 85.475)
+		(width 0.508)
+		(layer "B.Cu")
 		(net "/RX1")
 	)
 	(segment
-		(start 138.3 78.125)
-		(end 140.925 80.75)
-		(width 0.3)
-		(layer "F.Cu")
-		(net "/RX1")
-	)
-	(segment
-		(start 147.2 80.75)
-		(end 149.2 78.75)
-		(width 0.3)
-		(layer "F.Cu")
-		(net "/RX1")
-	)
-	(segment
-		(start 140.925 80.75)
-		(end 147.2 80.75)
-		(width 0.3)
-		(layer "F.Cu")
+		(start 147.2 88.1)
+		(end 140.925 88.1)
+		(width 0.508)
+		(layer "B.Cu")
 		(net "/RX1")
 	)
@@
 		(polygon
 			(pts
-				(xy 120.2 65.25) (xy 154.2 65.25) (xy 154.2 83.25) (xy 120.2 83.25)
-			)
-		)
+				(xy 120.2 65.25) (xy 154.2 65.25) (xy 154.2 90) (xy 120.2 90)
+			)
+		)
